File: ESP32_Personal_Health_Wearable/personal_health_wearable_v2/_autosave-personal_health_wearable_v2.kicad_sch (KiCad schematic)
At the start: 67 parts, among them J1 TYPE-C-31-M-12, J2 Conn_01x04_RA, J3 HLW5R-2C7LF, J4 JST_2mm_LiPo, SW1 SMD_4.6x2.8mm_h1.9mm, SW2 SMD_4.6x2.8mm_h1.9mm, U1 ESP32-C6-MINI-1, U2 USBLC6-2SC6, U3 TPS63001, U4 LMP91000SDE_NOPB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

Commit message: Completed schematic
Parts:
- added C33: 1.0uF, Capacitor_SMD:C_0402_1005Metric, symbol SparkFun-Capacitor:1.0uF_0402_16V_10%
Connections:
- net BIN: now also U1.19 (IO14)
- net GND: now also C32.2, C33.1
- net GPOUT: now also U1.20 (IO15)
- net VBATT: now also R15.1, U8.7 (SRN); no longer J4.2 (+), R15.2, U8.6 (BAT), U8.8 (SRP)
- net VDD: now also C32.1
- new net BATTERY: C33.2, J4.2 (+), R15.2, U8.6 (BAT), U8.8 (SRP)
- no-connect marks 10 -> 8

Commit message: Update _autosave-personal_health_wearable_v2.kicad_sch
Parts:
- J4: footprint PCM_SparkFun-Connector:JST_1x02_P2.0mm_Horizontal_SMD -> SparkFun-Connector:JST_1x02_P2.0mm_Horizontal_SMD
- R15: footprint PCM_SparkFun-Resistor:R_0402_1005Metric -> SparkFun-Resistor:R_0402_1005Metric
Connections:
- net ~{CHG}: now also U1.16 (IO7)
- net ~{PGOOD}: now also U1.15 (IO6)
- no-connect marks 8 -> 6
Changed lines of the file:
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@@
 	)
 	(junction
-		(at 339.09 109.22)
-		(diameter 0)
-		(color 0 0 0 0)
-	)
-	(junction
 		(at 195.58 64.77)
 		(diameter 0)
@@
 	)
 	(junction
+		(at 331.47 218.44)
+		(diameter 0)
+		(color 0 0 0 0)
+	)
+	(junction
 		(at 214.63 72.39)
 		(diameter 0)
@@
 	)
 	(no_connect
-		(at 68.58 62.23)
-	)
-	(no_connect
 		(at 35.56 222.25)
 	)
@@
 	)
 	(no_connect
-		(at 68.58 59.69)
-	)
-	(no_connect
 		(at 60.96 229.87)
 	)
@@
 	(wire
 		(pts
+			(xy 331.47 218.44) (xy 332.74 218.44)
+		)
+		(stroke
+			(width 0)
+			(type default)
+		)
+	)
+	(wire
+		(pts
 			(xy 87.63 33.02) (xy 90.17 33.02)
 		)
@@
 	(wire
 		(pts
-			(xy 339.09 109.22) (xy 330.2 109.22)
+			(xy 330.2 109.22) (xy 346.71 109.22)
 		)
 		(stroke
@@
 	(wire
 		(pts
-			(xy 328.93 218.44) (xy 332.74 218.44)
+			(xy 328.93 218.44) (xy 331.47 218.44)
 		)
 		(stroke
@@
 	(wire
 		(pts
-			(xy 346.71 109.22) (xy 339.09 109.22)
-		)
-		(stroke
-			(width 0)
-			(type default)
-		)
-	)
-	(wire
-		(pts
 			(xy 330.2 109.22) (xy 326.39 109.22)
 		)
@@
 		)
 	)
+	(label "~{CHG}"
+		(at 68.58 62.23 180)
+		(effects
+			(font
+				(size 1.27 1.27)
+			)
+			(justify right bottom)
+		)
+	)
 	(label "USBC.D+"
 		(at 118.11 49.53 0)
@@
 		)
 	)
+	(label "~{PGOOD}"
+		(at 68.58 59.69 180)
+		(effects
+			(font
+				(size 0.635 0.635)
+			)
+			(justify right bottom)
+		)
+	)
 	(label "WE2"
 		(at 35.56 224.79 0)
@@
 	)
 	(symbol
-		(lib_id "power:PWR_FLAG")
-		(at 339.09 109.22 0)
-		(unit 1)
-		(exclude_from_sim no)
-		(in_bom yes)
-		(on_board yes)
-		(dnp no)
-		(property "Reference" "#FLG01"
-			(at 339.09 107.315 0)
-			(effects
-				(font
-					(size 1.27 1.27)
-				)
-				(hide yes)
-			)
-		)
-		(property "Value" "PWR_FLAG"
-			(at 332.994 107.442 0)
-			(effects
-				(font
-					(size 0.635 0.635)
-				)
-				(justify left)
-			)
-		)
-		(property "Footprint" ""
-			(at 339.09 109.22 0)
-			(effects
-				(font
-					(size 1.27 1.27)
-				)
-				(hide yes)
-			)
-		)
-		(property "Datasheet" "~"
-			(at 339.09 109.22 0)
-			(effects
-				(font
-					(size 1.27 1.27)
-				)
-				(hide yes)
-			)
-		)
-		(property "Description" "Special symbol for telling ERC where power comes from"
-			(at 339.09 109.22 0)
-			(effects
-				(font
-					(size 1.27 1.27)
-				)
-				(hide yes)
-			)
-		)
-		(pin "1"
-		)
-		(instances
-			(project "personal_health_wearable_v2"
-				(path "/88216a86-3b04-4f00-b598-4a78937d00f1"
-					(reference "#FLG01")
-					(unit 1)
-				)
-			)
-		)
-	)
-	(symbol
 		(lib_id "power:GND")
 		(at 186.69 83.82 0)
@@
 			)
 		)
-		(property "Footprint" "PCM_SparkFun-Connector:JST_1x02_P2.0mm_Horizontal_SMD"
+		(property "Footprint" "SparkFun-Connector:JST_1x02_P2.0mm_Horizontal_SMD"
 			(at 316.23 229.87 0)
 			(effects
@@
 	)
 	(symbol
+		(lib_id "power:PWR_FLAG")
+		(at 331.47 218.44 0)
+		(unit 1)
+		(exclude_from_sim no)
+		(in_bom yes)
+		(on_board yes)
+		(dnp no)
+		(property "Reference" "#FLG01"
+			(at 331.47 216.535 0)
+			(effects
+				(font
+					(size 1.27 1.27)
+				)
+				(hide yes)
+			)
+		)
+		(property "Value" "PWR_FLAG"
+			(at 329.946 215.392 0)
+			(effects
+				(font
+					(size 0.635 0.635)
+				)
+				(justify left)
+			)
+		)
+		(property "Footprint" ""
+			(at 331.47 218.44 0)
+			(effects
+				(font
+					(size 1.27 1.27)
+				)
+				(hide yes)
+			)
+		)
+		(property "Datasheet" "~"
+			(at 331.47 218.44 0)
+			(effects
+				(font
+					(size 1.27 1.27)
+				)
+				(hide yes)
+			)
+		)
+		(property "Description" "Special symbol for telling ERC where power comes from"
+			(at 331.47 218.44 0)
+			(effects
+				(font
+					(size 1.27 1.27)
+				)
+				(hide yes)
+			)
+		)
+		(pin "1"
+		)
+		(instances
+			(project "personal_health_wearable_v2"
+				(path "/88216a86-3b04-4f00-b598-4a78937d00f1"
+					(reference "#FLG01")
+					(unit 1)
+				)
+			)
+		)
+	)
+	(symbol
 		(lib_id "SparkFun-Capacitor:1.0uF_0402_16V_10%")
 		(at 368.3 171.45 90)
@@
 			)
 		)
-		(property "Footprint" "PCM_SparkFun-Resistor:R_0402_1005Metric"
+		(property "Footprint" "SparkFun-Resistor:R_0402_1005Metric"
 			(at 329.692 232.41 0)
 			(effects
