File: ESP32_Personal_Health_Wearable/personal_health_wearable_v2/personal_health_wearable_v2.kicad_pcb (KiCad board)
At the start: 2 copper layers, 129.3 x 67.8 mm, 55 parts, among them J1 TYPE-C-31-M-12, J2 Conn_01x04_RA, J3 HLW5R-2C7LF, SW1 SMD_4.6x2.8mm_h1.9mm, SW2 SMD_4.6x2.8mm_h1.9mm, U1 ESP32-C6-MINI-1, U2 USBLC6-2SC6, U3 TPS63001, U4 LMP91000SDE_NOPB, U5 ADS1114IDGS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

Commit message: Completed design file, BoM, and Gerbers
Parts:
- removed R7: 0, Resistor_SMD:R_0402_1005Metric
- removed U2: USBLC6-2SC6, Package_TO_SOT_SMD:SOT-23-6
- added C29: 1.0uF, Capacitor_SMD:C_0402_1005Metric, F.Cu at (151.1, 102.7)
- added C30: 10uF, Capacitor_SMD:C_0402_1005Metric, F.Cu at (153.1, 106.5)
- added C31: 1.0uF, Capacitor_SMD:C_0402_1005Metric, F.Cu at (147.6, 106.5)
- added C32: 470nF, Capacitor_SMD:C_0402_1005Metric, F.Cu at (139.9, 105.0)
- added C33: 1.0uF, Capacitor_SMD:C_0402_1005Metric, F.Cu at (142.3, 107.4)
- added J4: JST_2mm_LiPo, SparkFun-Connector:JST_1x02_P2.0mm_Horizontal_SMD, F.Cu at (135.9, 110.5)
- added R11: 1.1K, Resistor_SMD:R_0402_1005Metric, F.Cu at (152.9, 104.4)
- added R12: 590, Resistor_SMD:R_0402_1005Metric, F.Cu at (149.5, 102.6)
- added R13: 10k, Resistor_SMD:R_0402_1005Metric, F.Cu at (148.5, 102.7)
- added R14: 10k, Resistor_SMD:R_0402_1005Metric, F.Cu at (148.2, 108.0)
- added R15: 0.01, SparkFun-Resistor:R_0402_1005Metric, F.Cu at (147.2, 104.5)
- added U7: BQ24075RGT, Package_DFN_QFN:VQFN-16-1EP_3x3mm_P0.5mm_EP1.6x1.6mm, F.Cu at (150.3, 105.8)
- added U8: BQ27441DRZR-G1A, Package_SON:Texas_S-PDSO-N12, F.Cu at (143.3, 104.4)
- moved SW1 81.9 mm to (140.0, 86.2)
- moved J3 81.3 mm to (132.9, 101.5), turned to -90 degrees
- moved SW2 75.8 mm to (164.4, 86.2)
- moved C12 75.7 mm to (130.7, 90.3), turned to 90 degrees
- moved D1 74.1 mm to (147.7, 99.7), turned to 90 degrees
- moved JP1 73.8 mm to (139.4, 122.9)
- moved C11 72.7 mm to (131.1, 96.2), turned to 90 degrees
- moved U5 70.0 mm to (140.4, 92.7)
- moved L2 68.9 mm to (156.3, 105.7), turned to 90 degrees
- moved C4 66.9 mm to (138.3, 88.2), turned to 180 degrees
- moved R10 65.0 mm to (136.4, 91.7), turned to 180 degrees
- moved U4 64.7 mm to (133.8, 88.8)
- moved U6 64.2 mm to (134.2, 94.8)
- moved C13 64.1 mm to (142.1, 95.0), turned to 180 degrees
- moved U3 63.1 mm to (160.8, 105.7)
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Connections:
- net Net-(U3-VIN) renamed VIN
- C11 pad 1: GND -> GNDA
- C12 pad 1: GND -> GNDA
- J2 pad 1: VUSB -> 3.3V
- U1 pad 15: unconnected-(U1-IO6-Pad15) -> /~{PGOOD}
- U1 pad 16: unconnected-(U1-IO7-Pad16) -> /~{CHG}
- U1 pad 17: /USB.D- -> /USBC.D-
- U1 pad 18: /USB.D+ -> /USBC.D+
- U1 pad 19: unconnected-(U1-IO14-Pad19) -> /BIN
- U1 pad 20: unconnected-(U1-IO15-Pad20) -> /GPOUT
Routing:
- net /BUSY: track 0.00 -> 59.4 mm, vias 0 -> 2
- net /RST: track 0.00 -> 53.7 mm, vias 0 -> 2
- net GND: track 0.00 -> 52.7 mm, vias 0 -> 12
- net 3.3V: track 0.00 -> 52.1 mm, vias 0 -> 12
- net /DC: track 0.00 -> 51.2 mm, vias 0 -> 2
- net /SCL: track 0.00 -> 49.0 mm, vias 0 -> 2
- net /CS: track 0.00 -> 41.7 mm, vias 0 -> 2
- net /CLK: track 0.00 -> 41.2 mm, vias 0 -> 2
- net /DIN: track 0.00 -> 41.1 mm, vias 0 -> 2
- net /SDA: track 0.00 -> 40.6 mm, vias 0 -> 3
- net /RE: track 0.00 -> 31.8 mm, vias 0 -> 2
- net /~{MENB_WE1}: track 0.00 -> 31.6 mm, vias 0 -> 2
- net 5V: track 0.00 -> 31.1 mm, vias 0 -> 2
- net /~{BOOT}: track 0.00 -> 27.3 mm, vias 0 -> 2
- net /~{MENB_WE2}: track 0.00 -> 26.5 mm, vias 0 -> 2
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- added copper zone on In2.Cu, net 3.3V
- added copper zone on B.Cu, net GND
- added copper zone on F.Cu, net GND
- added copper zone on In1.Cu, net GND
- added copper zone on In1.Cu, net GNDA
Other:
- board size 129.3 x 67.8 mm -> 47 x 47 mm
- copper layers 2 -> 4
