File: ESP32_Personal_Health_Wearable/personal_health_wearable_v2/personal_health_wearable_v2.kicad_sch (KiCad schematic)
At the start: 67 parts, among them J1 TYPE-C-31-M-12, J2 Conn_01x04_RA, J3 HLW5R-2C7LF, J4 JST_2mm_LiPo, SW1 SMD_4.6x2.8mm_h1.9mm, SW2 SMD_4.6x2.8mm_h1.9mm, U1 ESP32-C6-MINI-1, U2 USBLC6-2SC6, U3 TPS63001, U4 LMP91000SDE_NOPB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

Commit message: Completed design file, BoM, and Gerbers
Parts:
- removed R7: 0, Resistor_SMD:R_0402_1005Metric, symbol SparkFun-Resistor:0_0402
- removed U2: USBLC6-2SC6, Package_TO_SOT_SMD:SOT-23-6, symbol Power_Protection:USBLC6-2SC6
- added C33: 1.0uF, Capacitor_SMD:C_0402_1005Metric, symbol SparkFun-Capacitor:1.0uF_0402_16V_10%
- J4: footprint PCM_SparkFun-Connector:JST_1x02_P2.0mm_Horizontal_SMD -> SparkFun-Connector:JST_1x02_P2.0mm_Horizontal_SMD; LCSC (none) -> C295747
- R15: footprint PCM_SparkFun-Resistor:R_0402_1005Metric -> SparkFun-Resistor:R_0402_1005Metric
- R6: LCSC (none) -> C25076
- U8: LCSC (none) -> C473397
Connections:
- net USB.D+ is gone; now on net USBC.D+: U1.18 (IO13)
- net USB.D- is gone; now on net USBC.D-: U1.17 (IO12)
- net 3.3V: now also J2.1 (Pin_1)
- net BIN: now also U1.19 (IO14)
- net GND: now also C32.2, C33.1; no longer C11.1, C12.1
- net GNDA: now also C11.1, C12.1
- net GPOUT: now also U1.20 (IO15)
- net VBATT: now also R15.1, U8.7 (SRN); no longer J4.2 (+), R15.2, U8.6 (BAT), U8.8 (SRP)
- net VDD: now also C32.1
- net VUSB: no longer J2.1 (Pin_1)
- net ~{CHG}: now also U1.16 (IO7)
- net ~{PGOOD}: now also U1.15 (IO6)
- new net BATTERY: C33.2, J4.2 (+), R15.2, U8.6 (BAT), U8.8 (SRP)
- no-connect marks 10 -> 6
